File: psu_jaapg.sch (KiCad schematic (older format))
At the start: 36 parts, among them J1 Vin 16-24v, J2 Vout, Q1 2N3904, Q2 TIP142, U1 LM358, U2 LM358

Commit message: First etched version
Parts:
- added C4: 1uF, Capacitor_THT:CP_Radial_D5.0mm_P2.50mm, symbol Device:CP
- added C5: 10uF, Capacitor_THT:CP_Radial_D5.0mm_P2.50mm, symbol Device:CP
- added C6, C7: 22p, Capacitor_THT:C_Disc_D5.1mm_W3.2mm_P5.00mm, symbol Device:C
- added C8: 4.7uF, Capacitor_THT:CP_Radial_D5.0mm_P2.50mm, symbol Device:CP
- added H1, H2, H3, H4: MountingHole, MountingHole:MountingHole_4.3mm_M4, symbol Mechanical:MountingHole
- added MES2: Voltmeter_DC, Connector_PinHeader_2.54mm:PinHeader_1x02_P2.54mm_Vertical, symbol Device:Voltmeter_DC
- C1, C3: footprint (none) -> Capacitor_THT:C_Disc_D5.1mm_W3.2mm_P5.00mm
- C2: footprint (none) -> Capacitor_THT:CP_Radial_D16.0mm_P7.50mm
- D5, D7: footprint (none) -> Connector_PinHeader_2.54mm:PinHeader_1x02_P2.54mm_Vertical
- D6: footprint (none) -> Diode_THT:D_DO-35_SOD27_P10.16mm_Horizontal
- J1: value Vin 16-24v -> Vin 16-24v AC; footprint (none) -> TerminalBlock:TerminalBlock_Altech_AK300-2_P5.00mm
- J2: value Vout -> Vout 1-16v DC; footprint (none) -> TerminalBlock:TerminalBlock_Altech_AK300-2_P5.00mm
- Q1: footprint digikey-footprints:TO-92-3 -> Personal:TO-92_HandSolder_LongPads
- Q2: footprint digikey-footprints:TO-247-3 -> Connector_PinHeader_2.54mm:PinHeader_1x03_P2.54mm_Vertical
- R1, R2: value 2k2 -> 2k7; footprint (none) -> Resistor_THT:R_Axial_DIN0207_L6.3mm_D2.5mm_P10.16mm_Horizontal
- R10, R11, R12, R13, R14, R15, R16, R3, R4, R5, R7, R8, R9: footprint (none) -> Resistor_THT:R_Axial_DIN0207_L6.3mm_D2.5mm_P10.16mm_Horizontal
- R6: footprint (none) -> Resistor_THT:R_Axial_DIN0617_L17.0mm_D6.0mm_P20.32mm_Horizontal
- RV1, RV2: footprint (none) -> Connector_PinHeader_2.54mm:PinHeader_1x03_P2.54mm_Vertical
- RV3: footprint (none) -> Potentiometer_THT:Potentiometer_Runtron_RM-063_Horizontal
- U1, U2: footprint (none) -> Package_DIP:DIP-8_W7.62mm_LongPads
Connections:
- net GND: now also C4.2, C5.2, C8.2, MES2.1 (-)
- net at D6.1 (K), R14.1, R3.2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: now also C5.1
- net at RV1.2, U1.2 (-): now also C6.2
- net at R11.1, R12.2, U1.1: now also C6.1
- net at D8.1 (K), J2.1 (Pin_1), Q2.1 (E)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: now also C4.1, MES2.2 (+)
- net at Q1.2 (C), Q2.2 (B), R13.2: now also C8.1
- net at R13.1, U2.1: now also C7.2
- net at RV3.2, U2.2 (-): now also C7.1
Other:
- note added: "Current adjust"
- note added: "Optional cap:\ndelay V adjust\ncur. lim. is active"
- note added: "Voltage adjust"
- moved on the sheet: C1, C2, C3, D1, D2, D3, D4, D5, D6, D7, D8, J1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
