File: psu.kicad_pcb (KiCad board)
At the start: 2 copper layers, 90 x 60 mm, 55 parts, among them J1 Vin 16-24v AC, J2 Vout 1-16v DC, Q1 2N3904, Q2 TIP142, U1 LM358, U2 LM358

Commit message: Initial commit
Parts:
- removed the REF** at (142.2, 118.1)
- R14: value 10k -> 1k8
- R7: value 10k -> 1k
- RV1: value 50k -> 5k
- RV2: value 50k -> 10k
- moved R16 2.02 mm to (141.2, 121.3)
- moved RV3 2.02 mm to (146.3, 121.3)
- moved R15 1.44 mm to (164.5, 123.8)
- moved D7 1.40 mm to (150.5, 130.8)
Routing:
- net Net-(C8-Pad1): track 82.5 -> 96.2 mm
- net GND: track 154.5 -> 150.4 mm
- net Net-(C7-Pad1): track 52.9 -> 50.1 mm
- net Net-(Q1-Pad3): track 45.5 -> 44.5 mm
- net Net-(C4-Pad1): track 69.7 -> 68.9 mm
- net Net-(R15-Pad2): track 3.41 -> 4.08 mm
